File: VIC20_kbd.kicad_pcb (KiCad board)
At the start: 2 copper layers, 367.7 x 112.2 mm, 133 parts, among them J1 Conn_01x20, SW1 Key_1, SW10 Key_W, SW11 Key_R, SW12 Key_Y, SW13 Key_I, SW14 Key_P, SW15 Key_asterisk, SW16 Key_RETURN, SW17 Key_CTRL, SW18 Key_A, SW19 Key_D, SW2 Key_3, SW20 Key_G, SW21 Key_J, SW22 Key_L, SW23 Key_semicolon, SW24 Key_CRSRRIGHT, SW25 Key_STOP, SW26 Key_LSHFT, SW27 Key_X, SW28 Key_V, SW29 Key_N, SW3 Key_5, SW30 Key_comma, SW31 Key_slash, SW32 Key_CRSRDOWN, SW33 Key_SPACE, SW34 Key_Z, SW35 Key_C, SW36 Key_B, SW37 Key_M, SW38 Key_period, SW39 Key_RSHFT, SW4 Key_7, SW40 Key_F1, SW41 Key_CBM, SW42 Key_S, SW43 Key_F, SW44 Key_H, SW45 Key_K, SW46 Key_colon, SW47 Key_equals, SW48 Key_F3, SW49 Key_Q, SW5 Key_9, SW50 Key_E, SW51 Key_T, SW52 Key_U, SW53 Key_O, SW54 Key_at, SW55 Key_ARROWUP, SW56 Key_F5, SW57 Key_2, SW58 Key_4, SW59 Key_6, SW6 Key_Plus, SW60 Key_8, SW61 Key_0, SW62 Key_minus, SW63 Key_HOME, SW64 Key_F7, SW65 Key_SHFTLCK, SW66 Key_RESTORE, SW7 Key_Pound, SW8 Key_DEL, SW9 Key_ARROWLEFT

Commit message: Added rounded corners Added mounting holes and cables support holes
Parts:
- added REF**: MountingHole_2.2mm_M2, Mounting_Holes:MountingHole_2.2mm_M2, F.Cu at (148.5, 40.9)
- added REF**: MountingHole_2.2mm_M2, Mounting_Holes:MountingHole_2.2mm_M2, F.Cu at (-14.9, 151.2)
- added REF**: MountingHole_2.2mm_M2, Mounting_Holes:MountingHole_2.2mm_M2, F.Cu at (-14.9, 53.2)
- added REF**: MountingHole_2.2mm_M2, Mounting_Holes:MountingHole_2.2mm_M2, F.Cu at (296.0, 53.2)
- added REF**: MountingHole_2.2mm_M2, Mounting_Holes:MountingHole_2.2mm_M2, F.Cu at (85.6, 53.2)
- added REF**: MountingHole_2.2mm_M2, Mounting_Holes:MountingHole_2.2mm_M2, F.Cu at (190.7, 93.5)
- added REF**: MountingHole_2.2mm_M2, Mounting_Holes:MountingHole_2.2mm_M2, F.Cu at (113.7, 93.5)
- added REF**: MountingHole_2.2mm_M2, Mounting_Holes:MountingHole_2.2mm_M2, F.Cu at (161.0, 40.9)
- added REF**: MountingHole_2.2mm_M2, Mounting_Holes:MountingHole_2.2mm_M2, F.Cu at (173.7, 40.9)
- added REF**: MountingHole_2.2mm_M2, Mounting_Holes:MountingHole_2.2mm_M2, F.Cu at (186.4, 40.9)
- added REF**: MountingHole_2.2mm_M2, Mounting_Holes:MountingHole_2.2mm_M2, F.Cu at (199.1, 40.9)
- added REF**: MountingHole_2.2mm_M2, Mounting_Holes:MountingHole_2.2mm_M2, F.Cu at (346.2, 53.2)
- added REF**: MountingHole_2.2mm_M2, Mounting_Holes:MountingHole_2.2mm_M2, F.Cu at (346.2, 151.2)
- added REF**: MountingHole_2.2mm_M2, Mounting_Holes:MountingHole_2.2mm_M2, F.Cu at (193.4, 151.2)
- added REF**: MountingHole_2.2mm_M2, Mounting_Holes:MountingHole_2.2mm_M2, F.Cu at (48.0, 151.2)
Routing:
- net /RB: track 264.9 -> 255.7 mm
- net /RE: track 198.5 -> 194.7 mm
- net /C5: track 625.1 -> 627.1 mm
- net /R8: track 123.0 -> 124.9 mm
- net /RA: track 405.6 -> 403.8 mm
- net /C6: track 567.6 -> 569.3 mm
- net /C7: track 541.9 -> 543.6 mm
- net /RF: track 235.1 -> 233.7 mm
- net /C4: track 593.8 -> 595.2 mm
- net /C3: track 698.0 -> 699.3 mm
- net /C2: track 495.5 -> 496.7 mm
- net /RC: track 199.0 -> 198.5 mm
Other:
- board size 367.7 x 112.2 mm -> 367.7 x 117.2 mm
- board text added: "VIC-20 keyboard for Cherry MX switches. V1.1 June 2019, Hans@Liss.nu"

Commit message: Rerouted everything, tidier V1.2
Parts:
- added REF**: MountingHole_2.2mm_M2, Mounting_Holes:MountingHole_2.2mm_M2, F.Cu at (93.2, 149.3)
- added REF**: MountingHole_2.2mm_M2, Mounting_Holes:MountingHole_2.2mm_M2, F.Cu at (145.2, 149.3)
- added REF**: MountingHole_2.2mm_M2, Mounting_Holes:MountingHole_2.2mm_M2, F.Cu at (296.9, 134.4)
- moved REF** 20.8 mm to (84.9, 74.0)
- moved REF** 18.0 mm to (187.1, 134.4)
- moved REF** 17.3 mm to (52.1, 134.4)
- moved REF** 13.4 mm to (304.2, 63.8)
- moved REF** 3.77 mm to (345.8, 57.0)
- moved REF** 3.76 mm to (-14.7, 57.0)
- moved REF** 1.99 mm to (345.8, 149.3)
- moved REF** 1.97 mm to (-14.7, 149.3)
Routing:
- net /C3: track 699.3 -> 504.1 mm, vias 8 -> 0
- net /C1: track 535.4 -> 404.0 mm, vias 7 -> 2
- net /C7: track 543.6 -> 414.8 mm, vias 3 -> 2
- net /C5: track 627.1 -> 558.4 mm, vias 5 -> 3
- net /C6: track 569.3 -> 504.1 mm, vias 6 -> 0
- net /C2: track 496.7 -> 432.8 mm, vias 9 -> 0
- net /RH: track 379.0 -> 330.6 mm, vias 2 -> 1
- net /C4: track 595.2 -> 554.4 mm
- net /C0: track 326.5 -> 306.8 mm, vias 1 -> 0
- net /RA: track 403.8 -> 419.4 mm
- net /RG: track 283.7 -> 269.1 mm, vias 4 -> 1
- net /R8: track 124.9 -> 115.7 mm
- net /RC: track 198.5 -> 204.2 mm
- net /RB: track 255.7 -> 259.1 mm
- net /RI: track 115.7 -> 119.1 mm
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Other:
- board size 367.7 x 117.2 mm -> 367.7 x 116.2 mm
- board text added: "VIC-20 keyboard for Cherry MX switches. V1.2 June 2019, Hans@Liss.nu"
- board text removed: "VIC-20 keyboard for Cherry MX switches. V1.1 June 2019, Hans@Liss.nu"

Commit message: Added SHIFT LOCK flip-flop to PCB Added Gerber files
Parts:
- removed D66: D, Diodes_SMD:D_0603
- added C1: 1uF, Capacitors_SMD:C_0603, F.Cu at (15.4, 136.2)
- added C2: 1uF, Capacitors_SMD:C_0603, F.Cu at (9.95, 134.7)
- added Q1: BC548, TO_SOT_Packages_SMD:SOT-23, F.Cu at (25.6, 136.0)
- added R1: 100k, Resistors_SMD:R_0603, F.Cu at (19.7, 136.2)
- added R2: 1k, Resistors_SMD:R_0603, F.Cu at (22.4, 140.1)
- added R3: 10k, Resistors_SMD:R_0603, F.Cu at (22.1, 136.2)
- added R4: 10k, Resistors_SMD:R_0603, F.Cu at (17.5, 140.2)
- added R5: 390, Resistors_SMD:R_0603, F.Cu at (17.4, 136.2)
- added R6: 10k, Resistors_SMD:R_0603, F.Cu at (6.16, 134.6)
- added REF**: MountingHole_3mm_M3, Mounting_Holes:MountingHole_3.2mm_M3, F.Cu at (61.1, 135.2)
- added REF**: MountingHole_3mm_M3, Mounting_Holes:MountingHole_3.2mm_M3, F.Cu at (186.1, 135.2)
- added REF**: MountingHole_4mm, Mounting_Holes:MountingHole_4mm, F.Cu at (186.1, 150.4)
- added REF**: MountingHole_4mm, Mounting_Holes:MountingHole_4mm, F.Cu at (61.1, 150.4)
- added U1: LM555, Housings_SOIC:SOIC-8_3.9x4.9mm_Pitch1.27mm, F.Cu at (8.97, 140.0)
- D65: value D -> LED; footprint Diodes_SMD:D_0603 -> LEDs:LED_D5.0mm; moved to F.Cu
- moved D65 20.6 mm to (5.97, 114.1), turned to 0 degrees
- moved REF** 6.36 mm to (193.4, 134.4)
- moved D33 3.00 mm to (129.1, 137.1)
- moved SW33 3.00 mm to (126.2, 137.1)
- moved D56 1.19 mm to (337.1, 99.3)
- moved D64 1.19 mm to (337.1, 118.6)
- moved D48 1.15 mm to (337.1, 80.0)
- moved SW56 1.09 mm to (333.9, 99.3)
- moved SW64 1.09 mm to (333.9, 118.6)
- moved SW48 1.04 mm to (333.9, 80.0)
- moved D40 1.00 mm to (337.1, 60.7)
- moved SW40 1.00 mm to (333.9, 60.7)
Connections:
- D65 pad 1: /RA -> GND
- J1 pad 1: /RI -> GND
- J1 pad 4: (no net) -> VCC
- SW65 pad 1: Net-(D65-Pad2) -> Net-(C1-Pad1)
- SW65 pad 2: /C1 -> Net-(R3-Pad1)
- SW66 pad 1: Net-(D66-Pad2) -> GND
Routing:
- net GND: track 0.00 -> 510.5 mm, vias 0 -> 3
- net VCC: track 0.00 -> 345.0 mm, vias 0 -> 2
- net /RI: track 119.1 -> 0.00 mm
- net Net-(R3-Pad1): track 0.00 -> 69.7 mm, vias 0 -> 5
- net Net-(C1-Pad1): track 0.00 -> 56.8 mm, vias 0 -> 1
- net /C1: track 404.0 -> 362.4 mm
- net Net-(D65-Pad2): track 2.16 -> 27.6 mm, vias 0 -> 3
- net Net-(D26-Pad2): track 2.17 -> 27.5 mm, vias 0 -> 1
- net /C3: track 504.1 -> 519.5 mm
- net Net-(R1-Pad1): track 0.00 -> 13.7 mm, vias 0 -> 2
- net Net-(C2-Pad1): track 0.00 -> 8.43 mm, vias 0 -> 2
- net /C4: track 554.4 -> 558.8 mm
- net Net-(Q1-Pad1): track 0.00 -> 4.08 mm
- net /C5: track 558.4 -> 561.7 mm
- net /C6: track 504.1 -> 507.2 mm
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Other:
- board text added: "VIC-20 keyboard for Cherry MX switches. V1.3 August 2019, Hans@Liss.nu"
- board text removed: "VIC-20 keyboard for Cherry MX switches. V1.2 June 2019, Hans@Liss.nu"

Commit message: Cleaned up to accommodate Kailh sockets.
Parts:
- moved Q1 7.93 mm to (19.8, 141.4)
- moved R5 7.93 mm to (11.6, 141.6)
- moved R6 7.93 mm to (0.34, 140.0)
- moved C2 7.93 mm to (4.13, 140.1)
- moved C1 7.93 mm to (9.59, 141.5)
- moved R1 7.93 mm to (13.9, 141.5)
- moved R2 7.93 mm to (16.5, 145.4)
- moved R3 7.93 mm to (16.3, 141.5)
- moved R4 7.93 mm to (11.7, 145.5)
- moved U1 7.93 mm to (3.15, 145.3)
Routing:
- net /C3: track 519.5 -> 604.6 mm, vias 0 -> 1
- net /C2: track 432.8 -> 505.7 mm
- net /C7: track 414.7 -> 475.5 mm
- net /C1: track 362.4 -> 397.1 mm, vias 2 -> 1
- net GND: track 510.5 -> 485.1 mm, vias 3 -> 4
- net /C4: track 558.8 -> 580.4 mm, vias 2 -> 1
- net /C5: track 561.7 -> 578.7 mm, vias 3 -> 2
- net Net-(C1-Pad1): track 56.8 -> 73.7 mm
- net Net-(R3-Pad1): track 69.7 -> 85.0 mm, vias 5 -> 1
- net /RA: track 421.5 -> 409.8 mm, vias 0 -> 1
- net /RG: track 269.4 -> 277.9 mm
- net /RE: track 197.3 -> 205.7 mm
- net /RF: track 230.3 -> 238.6 mm
- net VCC: track 345.0 -> 337.2 mm
- net /C6: track 507.2 -> 514.8 mm, vias 0 -> 2
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
Commit message: Cleaned up SHIFT LOCK area and fixed silkscreen.
Other:
- board text added: "SHIFT LOCK"
- board text added: "VIC-20 keyboard for Cherry MX switches. V2.0 January 2021, Hans@Liss.nu"
- board text removed: "VIC-20 keyboard for Cherry MX switches. V1.3 August 2019, Hans@Liss.nu"
Changed lines of the file:
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@@
   (general
     (thickness 1.6)
-    (drawings 33)
+    (drawings 39)
     (tracks 1268)
     (zones 0)
@@
     (tags "resistor 0603")
     (attr smd)
-    (fp_text reference R6 (at 0 -1.45) (layer F.SilkS)
+    (fp_text reference R6 (at -0.02 1.44) (layer F.SilkS)
       (effects (font (size 1 1) (thickness 0.15)))
     )
-    (fp_text value 10k (at 0 1.5) (layer F.Fab)
+    (fp_text value 10k (at 0.05 -1.58) (layer F.SilkS)
       (effects (font (size 1 1) (thickness 0.15)))
     )
@@
     (tags "capacitor 0603")
     (attr smd)
-    (fp_text reference C2 (at 0 -1.5) (layer F.SilkS)
+    (fp_text reference C2 (at -0.07 1.51) (layer F.SilkS)
       (effects (font (size 1 1) (thickness 0.15)))
     )
-    (fp_text value 1uF (at 0 1.5) (layer F.Fab)
+    (fp_text value 1uF (at 0.21 -1.72) (layer F.SilkS)
       (effects (font (size 1 1) (thickness 0.15)))
     )
@@
     (tags "capacitor 0603")
     (attr smd)
-    (fp_text reference C1 (at 0 -1.5 90) (layer F.SilkS)
+    (fp_text reference C1 (at 2.14 -0.11) (layer F.SilkS)
       (effects (font (size 1 1) (thickness 0.15)))
     )
-    (fp_text value 1uF (at 0 1.5 90) (layer F.Fab)
+    (fp_text value 1uF (at -3 0.14 270) (layer F.SilkS)
       (effects (font (size 1 1) (thickness 0.15)))
     )
@@
     (tags SOT-23)
     (attr smd)
-    (fp_text reference Q1 (at 0 -2.5 90) (layer F.SilkS)
+    (fp_text reference Q1 (at -2.68 0.03 180) (layer F.SilkS)
       (effects (font (size 1 1) (thickness 0.15)))
     )
-    (fp_text value BC548 (at 0 2.5 90) (layer F.Fab)
+    (fp_text value BC548 (at 0 2.5 90) (layer F.SilkS)
       (effects (font (size 1 1) (thickness 0.15)))
     )
@@
     (tags "resistor 0603")
     (attr smd)
-    (fp_text reference R1 (at 0 -1.45 90) (layer F.SilkS)
+    (fp_text reference R1 (at -2.08 -0.01 180) (layer F.SilkS)
       (effects (font (size 1 1) (thickness 0.15)))
     )
-    (fp_text value 100k (at 0 1.5 90) (layer F.Fab)
+    (fp_text value 100k (at 3.46 -0.17 90) (layer F.SilkS)
       (effects (font (size 1 1) (thickness 0.15)))
     )
@@
       (effects (font (size 1 1) (thickness 0.15)))
     )
-    (fp_text value 1k (at 0 1.5) (layer F.Fab)
+    (fp_text value 1k (at -2.47 -0.1) (layer F.SilkS)
       (effects (font (size 1 1) (thickness 0.15)))
     )
@@
     (tags "resistor 0603")
     (attr smd)
-    (fp_text reference R3 (at 0 -1.45 90) (layer F.SilkS)
+    (fp_text reference R3 (at 2.11 -0.06 180) (layer F.SilkS)
       (effects (font (size 1 1) (thickness 0.15)))
     )
-    (fp_text value 10k (at 0 1.5 90) (layer F.Fab)
+    (fp_text value 10k (at -3 -0.03 90) (layer F.SilkS)
       (effects (font (size 1 1) (thickness 0.15)))
     )
@@
     (tags "resistor 0603")
     (attr smd)
-    (fp_text reference R4 (at 0 -1.45 90) (layer F.SilkS)
+    (fp_text reference R4 (at 2.06 -0.06 180) (layer F.SilkS)
       (effects (font (size 1 1) (thickness 0.15)))
     )
-    (fp_text value 10k (at 0 1.5 90) (layer F.Fab)
+    (fp_text value 10k (at 0.13 1.5 90) (layer F.SilkS)
       (effects (font (size 1 1) (thickness 0.15)))
     )
@@
     (tags "resistor 0603")
     (attr smd)
-    (fp_text reference R5 (at 0 -1.45 90) (layer F.SilkS)
+    (fp_text reference R5 (at -2.04 0.02 180) (layer F.SilkS)
       (effects (font (size 1 1) (thickness 0.15)))
     )
-    (fp_text value 390 (at 0 1.5 90) (layer F.Fab)
+    (fp_text value 390 (at 3.22 0.12 90) (layer F.SilkS)
       (effects (font (size 1 1) (thickness 0.15)))
     )
@@
     (tags "SOIC 1.27")
     (attr smd)
-    (fp_text reference U1 (at 0 -3.5) (layer F.SilkS)
+    (fp_text reference U1 (at 0.02 -3.65) (layer F.SilkS)
       (effects (font (size 1 1) (thickness 0.15)))
     )
-    (fp_text value LM555 (at 0 3.5) (layer F.Fab)
+    (fp_text value LM555 (at -0.1 -5.05) (layer F.SilkS)
       (effects (font (size 1 1) (thickness 0.15)))
     )
@@
     )
   )
-  (gr_text "VIC-20 keyboard for Cherry MX switches. V1.3\nAugust 2019, Hans@Liss.nu" (at 304.25 147.9) (layer F.SilkS)
+  (gr_line (start 15.38 149.16) (end 15.38 151.11) (layer F.SilkS) (width 0.15))
+  (gr_line (start 24.65 149.16) (end 15.38 149.16) (layer F.SilkS) (width 0.15))
+  (gr_text "SHIFT LOCK" (at 20 150.12) (layer F.SilkS)
+    (effects (font (size 1 1) (thickness 0.15)))
+  )
+  (gr_line (start -4.28 151.12) (end -4.29 136.04) (layer F.SilkS) (width 0.15))
+  (gr_line (start 24.58 151.12) (end -4.28 151.12) (layer F.SilkS) (width 0.15))
+  (gr_line (start 24.67 136.02) (end 24.64 151.12) (layer F.SilkS) (width 0.15))
+  (gr_line (start -4.28 136.02) (end 24.67 136.02) (layer F.SilkS) (width 0.15))
+  (gr_text "VIC-20 keyboard for Cherry MX switches. V2.0\nJanuary 2021, Hans@Liss.nu" (at 304.25 147.9) (layer F.SilkS)
     (effects (font (size 1.5 1.5) (thickness 0.3)))
   )
@@
   (gr_line (start 37.4 152.76) (end 210.4 152.76) (angle 90) (layer F.SilkS) (width 0.2))
   (gr_line (start 37.4 133.76) (end 37.4 152.76) (angle 90) (layer F.SilkS) (width 0.2))
-  (gr_line (start -20.42 139.15) (end 31.58 139.15) (angle 90) (layer F.SilkS) (width 0.2))
   (gr_line (start -14.57 104.24) (end -14.57 104.26) (angle 90) (layer F.SilkS) (width 0.2))
   (gr_line (start -14.63 104.24) (end -14.57 104.24) (angle 90) (layer F.SilkS) (width 0.2))

Commit message: Additional preparation for Kailh sockets
Parts:
- moved C1 80.8 mm to (54.1, 209.0)
- moved D10 80.8 mm to (96.7, 146.9)
- moved D18 80.8 mm to (83.3, 166.1)
- moved D24 80.8 mm to (332.7, 185.3)
- moved D25 80.8 mm to (44.9, 166.1)
- moved D26 80.8 mm to (68.8, 185.3)
- moved D27 80.8 mm to (111.9, 185.3)
- moved D28 80.8 mm to (150.4, 185.3)
- moved D29 80.8 mm to (188.8, 185.3)
- moved D30 80.8 mm to (227.1, 185.3)
- moved D31 80.8 mm to (265.6, 185.3)
- moved D32 80.8 mm to (313.5, 185.3)
- moved D33 80.8 mm to (173.6, 204.5)
- moved D34 80.8 mm to (92.7, 185.3)
- moved D36 80.8 mm to (169.6, 185.3)
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Routing:
- net /RE: track 205.7 -> 214.4 mm
- net /RA: track 409.8 -> 418.4 mm
- net /C4: track 580.4 -> 585.9 mm
- net /RD: track 189.2 -> 194.3 mm
- net Net-(D26-Pad2): track 34.1 -> 38.7 mm
- net /C2: track 505.7 -> 510.2 mm
- net /C1: track 397.1 -> 401.2 mm
- net /RB: track 265.4 -> 269.3 mm
- net /C3: track 604.6 -> 608.2 mm
- net /C6: track 514.8 -> 518.0 mm
- net /C5: track 578.7 -> 581.6 mm
- net GND: track 485.1 -> 483.5 mm
- net /RG: track 277.9 -> 279.4 mm
- net /RH: track 333.5 -> 332.6 mm

Commit message: Kailh sockets A big diode symbol on bottom silkscreen layer, as a guide.
Parts:
- SW1, SW10, SW11, SW12, SW13, SW14, SW15, SW18, SW19, SW2, SW20, SW21, SW22, SW23, SW24, SW25, SW27, SW28, SW29, SW3, SW30, SW31, SW32, SW34, SW35, SW36, SW37, SW38, SW4, SW41, SW42, SW43, SW44, SW45, SW46, SW47, SW49, SW5, SW50, SW51, SW52, SW53, SW54, SW55, SW57, SW58, SW59, SW6, SW60, SW61, SW62, SW63, SW65, SW7, SW8, SW9: footprint Buttons_Switches_Keyboard:SW_Cherry_MX1A_1.00u_PCB -> keyswitches:Kailh_socket_MX_optional_compatible
- SW16: footprint Buttons_Switches_Keyboard:SW_Cherry_MX1A_2.00u_PCB -> keyswitches:Kailh_socket_MX_optional_compatible
- SW17, SW26, SW39, SW40, SW48, SW56, SW64, SW66: footprint Buttons_Switches_Keyboard:SW_Cherry_MX1A_1.50u_PCB -> keyswitches:Kailh_socket_MX_optional_compatible
- SW33: footprint Buttons_Switches_Keyboard:SW_Cherry_MX1A_6.25u_PCB -> keyswitches:Kailh_socket_MX_optional_compatible
Routing:
- net /C0: track 306.8 -> 381.8 mm
- net /C1: track 401.2 -> 475.2 mm
- net /C5: track 581.6 -> 655.3 mm
- net /C2: track 510.2 -> 583.8 mm
- net /C6: track 518.0 -> 591.4 mm
- net /C3: track 608.2 -> 681.6 mm
- net /C7: track 475.5 -> 548.7 mm
- net /C4: track 585.9 -> 634.5 mm, vias 1 -> 2
- net /RH: track 332.6 -> 346.5 mm
- net Net-(D53-Pad2): track 2.22 -> 16.0 mm, vias 0 -> 2
- net GND: track 483.5 -> 495.0 mm
- net Net-(C1-Pad1): track 73.2 -> 83.8 mm
- net Net-(D5-Pad2): track 2.19 -> 12.5 mm, vias 0 -> 2
- net Net-(R3-Pad1): track 84.6 -> 93.7 mm
- net /R8: track 115.7 -> 124.8 mm
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